Commit message: add wheels to robot

File: src/my_robot/urdf/my_robot.xacro (robot description, xacro)
@@ -54,3 +54,65 @@
     </visual>
   </link>
+  <link name='left_wheel'>
+    <inertial>
+      <mass value="5.0"/>
+      <origin xyz="0.0 0 0" rpy="0 1.5707 1.5707"/>
+      <inertia
+          ixx="0.1" ixy="0" ixz="0"
+          iyy="0.1" iyz="0"
+          izz="0.1"
+      />
+    </inertial>
+    <collision name='left_wheel_collision'>
+      <origin xyz="0 0 0" rpy="0 1.5707 1.5707"/>
+      <geometry>
+        <cylinder radius=".1" length=".05"/>
+      </geometry>
+    </collision>
+    <visual name='left_wheel_visual'>
+      <origin xyz="0 0 0" rpy="0 1.5707 1.5707"/>
+      <geometry>
+        <cylinder radius=".1" length=".05"/>
+      </geometry>
+    </visual>
+  </link>
+  <link name='right_wheel'>
+    <inertial>
+      <mass value="5.0"/>
+      <origin xyz="0.0 0 0" rpy="0 1.5707 1.5707"/>
+      <inertia
+          ixx="0.1" ixy="0" ixz="0"
+          iyy="0.1" iyz="0"
+          izz="0.1"
+      />
+    </inertial>
+    <collision name='right_wheel_collision'>
+      <origin xyz="0 0 0" rpy="0 1.5707 1.5707"/>
+      <geometry>
+        <cylinder radius=".1" length=".05"/>
+      </geometry>
+    </collision>
+    <visual name='right_wheel_visual'>
+      <origin xyz="0 0 0" rpy="0 1.5707 1.5707"/>
+      <geometry>
+        <cylinder radius=".1" length=".05"/>
+      </geometry>
+    </visual>
+  </link>
+  <joint type="continuous" name="left_wheel_hinge">
+    <origin xyz="0 0.15 0" rpy="0 0 0"/>
+    <child link="left_wheel"/>
+    <parent link="chassis"/>
+    <axis xyz="0 1 0" rpy="0 0 0"/>
+    <limit effort="10000" velocity="1000"/>
+    <dynamics damping="1.0" friction="1.0"/>
+  </joint>
+  <joint type="continuous" name="right_wheel_hinge">
+    <origin xyz="0 -0.15 0" rpy="0 0 0"/>
+    <child link="right_wheel"/>
+    <parent link="chassis"/>
+    <axis xyz="0 1 0" rpy="0 0 0"/>
+    <limit effort="10000" velocity="1000"/>
+    <dynamics damping="1.0" friction="1.0"/>
+  </joint>
 </robot>

Commit message: add camera to robot

File: src/my_robot/urdf/my_robot.xacro (robot description, xacro)
@@ -100,4 +100,30 @@
     </visual>
   </link>
+  <link name='camera'>
+    <inertial>
+      <mass value=".1"/>
+      <origin xyz="0.0 0 0" rpy="0 0 0"/>
+      <box_inertia
+          m=".1" x=".05" y=".05" z=".05"
+      />
+      <inertia
+          ixx="1e-6" ixy="0" ixz="0"
+          iyy="1e-6" iyz="0"
+          izz="1e-6"
+      />
+    </inertial>
+    <collision name='camera_collision'>
+      <origin xyz="0 0 0" rpy="0 0 0"/>
+      <geometry>
+        <box size= ".05 .05 .05"/>
+      </geometry>
+    </collision>
+    <visual name='camera_visual'>
+      <origin xyz="0 0 0" rpy="0 1.5707 1.5707"/>
+      <geometry>
+        <box size= ".05 .05 .05"/>
+      </geometry>
+    </visual>
+  </link>
   <joint type="continuous" name="left_wheel_hinge">
     <origin xyz="0 0.15 0" rpy="0 0 0"/>
@@ -116,3 +142,9 @@
     <dynamics damping="1.0" friction="1.0"/>
   </joint>
+  <joint type="fixed" name="camera_joint">
+    <origin xyz=".2 0 0" rpy="0 0 0"/>
+    <child link="camera"/>
+    <parent link="chassis"/>
+    <axis xyz="0 1 0" rpy="0 0 0"/>
+  </joint>
 </robot>

Commit message: add lidar to robot

File: src/my_robot/urdf/my_robot.xacro (robot description, xacro)
@@ -120,7 +120,33 @@
     </collision>
     <visual name='camera_visual'>
-      <origin xyz="0 0 0" rpy="0 1.5707 1.5707"/>
+      <origin xyz="0 0 0" rpy="0 0 0"/>
       <geometry>
         <box size= ".05 .05 .05"/>
+      </geometry>
+    </visual>
+  </link>
+  <link name='hokuyo'>
+    <inertial>
+      <mass value="1e-5"/>
+      <origin xyz="0.0 0 0" rpy="0 0 0"/>
+      <box_inertia
+          m=".1" x=".05" y=".05" z=".05"
+      />
+      <inertia
+          ixx="1e-6" ixy="0" ixz="0"
+          iyy="1e-6" iyz="0"
+          izz="1e-6"
+      />
+    </inertial>
+    <collision name='hokuyo_collision'>
+      <origin xyz="0 0 0" rpy="0 0 0"/>
+      <geometry>
+        <box size= ".1 .1 .1"/>
+      </geometry>
+    </collision>
+    <visual name='hokuyo_visual'>
+      <origin xyz="0 0 0" rpy="0 0 0"/>
+      <geometry>
+        <filename = “package://my_robot/meshes/hokuyo.dae”/>
       </geometry>
     </visual>
@@ -148,3 +174,9 @@
     <axis xyz="0 1 0" rpy="0 0 0"/>
   </joint>
+  <joint type="fixed" name="hokuyo_joint">
+    <origin xyz=".15 0 .1" rpy="0 0 0"/>
+    <child link="camera"/>
+    <parent link="hokuyo"/>
+    <axis xyz="0 1 0" rpy="0 0 0"/>
+  </joint>
 </robot>

Commit message: add meshes and color

File: src/my_robot/urdf/my_robot.xacro (robot description, xacro)
@@ -180,3 +180,6 @@
     <axis xyz="0 1 0" rpy="0 0 0"/>
   </joint>
+  <gazebo reference="left_wheel">
+      <material>Gazebo/Green</material>
+  </gazebo>
 </robot>

Commit message: fixes in my_robot.xacro

File: src/my_robot/urdf/my_robot.xacro (robot description, xacro)
@@ -130,7 +130,4 @@
       <mass value="1e-5"/>
       <origin xyz="0.0 0 0" rpy="0 0 0"/>
-      <box_inertia
-          m=".1" x=".05" y=".05" z=".05"
-      />
       <inertia
           ixx="1e-6" ixy="0" ixz="0"
@@ -148,5 +145,5 @@
       <origin xyz="0 0 0" rpy="0 0 0"/>
       <geometry>
-        <filename = “package://my_robot/meshes/hokuyo.dae”/>
+        <mesh filename="package://my_robot/meshes/hokuyo.dae"/>
       </geometry>
     </visual>
@@ -176,10 +173,10 @@
   <joint type="fixed" name="hokuyo_joint">
     <origin xyz=".15 0 .1" rpy="0 0 0"/>
-    <child link="camera"/>
-    <parent link="hokuyo"/>
+    <child link="hokuyo"/>
+    <parent link="chassis"/>
     <axis xyz="0 1 0" rpy="0 0 0"/>
   </joint>
   <gazebo reference="left_wheel">
-      <material>Gazebo/Green</material>
+    <material>Gazebo/Green</material>
   </gazebo>
 </robot>
